File: upd78214-breakout.kicad_sch (KiCad schematic)
At the start: 9 parts, among them J1 Conn_02x17_Odd_Even, U1 upd78214-64p-qfp, X1 USB-B1HSB6

Commit message: Refresh info
Parts:
- gave numbers to parts that had none: 2
Changed lines of the file:
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@@
   (symbol (lib_id "Device:R_Small_US") (at 27.94 63.5 90) (unit 1)
     (in_bom yes) (on_board yes) (fields_autoplaced)
-    (property "Reference" "R?" (id 0) (at 27.94 57.15 90))
+    (property "Reference" "R3" (id 0) (at 27.94 57.15 90))
     (property "Value" "1kΩ" (id 1) (at 27.94 59.69 90))
     (property "Footprint" "Resistor_THT:R_Axial_DIN0207_L6.3mm_D2.5mm_P10.16mm_Horizontal" (id 2) (at 27.94 63.5 0)
@@
   (symbol (lib_id "power:GND") (at 46.99 73.025 0) (unit 1)
     (in_bom yes) (on_board yes) (fields_autoplaced)
-    (property "Reference" "#PWR?" (id 0) (at 46.99 79.375 0)
+    (property "Reference" "#PWR0108" (id 0) (at 46.99 79.375 0)
       (effects (font (size 1.27 1.27)) hide)
     )
@@
   (symbol (lib_id "power:+5V") (at 18.415 53.34 0) (unit 1)
     (in_bom yes) (on_board yes) (fields_autoplaced)
-    (property "Reference" "#PWR?" (id 0) (at 18.415 57.15 0)
+    (property "Reference" "#PWR0106" (id 0) (at 18.415 57.15 0)
       (effects (font (size 1.27 1.27)) hide)
     )
@@
   (symbol (lib_id "Device:LED") (at 35.56 63.5 180) (unit 1)
     (in_bom yes) (on_board yes) (fields_autoplaced)
-    (property "Reference" "D?" (id 0) (at 37.1475 55.88 0))
+    (property "Reference" "D1" (id 0) (at 37.1475 55.88 0))
     (property "Value" "LED" (id 1) (at 37.1475 58.42 0))
     (property "Footprint" "LED_THT:LED_D3.0mm" (id 2) (at 35.56 63.5 0)
@@
       (reference "#PWR0105") (unit 1) (value "GND") (footprint "")
     )
+    (path "/c23ff1c5-20c9-4736-876c-63fbe66acba4"
+      (reference "#PWR0106") (unit 1) (value "+5V") (footprint "")
+    )
     (path "/8859959c-fd90-4c08-9c36-a742ed7339e5"
       (reference "#PWR0107") (unit 1) (value "GND") (footprint "")
     )
     (path "/70fd9e4d-9828-4147-abe2-fb3e729fec4d"
-      (reference "#PWR?") (unit 1) (value "GND") (footprint "")
-    )
-    (path "/c23ff1c5-20c9-4736-876c-63fbe66acba4"
-      (reference "#PWR?") (unit 1) (value "+5V") (footprint "")
+      (reference "#PWR0108") (unit 1) (value "GND") (footprint "")
     )
     (path "/ea05f697-d9aa-459a-811b-0d351998e19b"
-      (reference "D?") (unit 1) (value "LED") (footprint "LED_THT:LED_D3.0mm")
+      (reference "D1") (unit 1) (value "LED") (footprint "LED_THT:LED_D3.0mm")
     )
     (path "/bc0e9206-078d-474c-ade8-99441c6f82a5"
@@
     )
     (path "/442545a2-72ff-41c0-aa0b-a97b9106ee1b"
-      (reference "R?") (unit 1) (value "1kΩ") (footprint "Resistor_THT:R_Axial_DIN0207_L6.3mm_D2.5mm_P10.16mm_Horizontal")
+      (reference "R3") (unit 1) (value "1kΩ") (footprint "Resistor_THT:R_Axial_DIN0207_L6.3mm_D2.5mm_P10.16mm_Horizontal")
     )
     (path "/b3494da2-9112-497d-8dd3-ab62d10d763a"

Commit message: Break out NMI pin
Connections:
- net PROG_NMI: now reaches U1.28 (p2,0/nmi)
- net PROG_NMI: now also J1.22 (Pin_22)
- no-connect marks 8 -> 7
Changed lines of the file:
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@@
   (no_connect (at 51.435 114.3))
   (no_connect (at 51.435 116.84))
-  (no_connect (at 51.435 119.38))
   (no_connect (at 51.435 109.22))
   (no_connect (at 51.435 106.68))
@@
     (stroke (width 0) (type default) (color 0 0 0 0))
   )
+  (wire (pts (xy 103.505 57.15) (xy 111.125 57.15))
+    (stroke (width 0) (type default) (color 0 0 0 0))
+  )
   (wire (pts (xy 103.505 113.03) (xy 111.125 113.03))
     (stroke (width 0) (type default) (color 0 0 0 0))
@@
     (effects (font (size 1.27 1.27)) (justify left bottom))
   )
+  (label "PROG_NMI" (at 51.435 119.38 0)
+    (effects (font (size 1.27 1.27)) (justify left bottom))
+  )
   (label "PROG_D7" (at 111.125 118.11 0)
     (effects (font (size 1.27 1.27)) (justify left bottom))
@@
     (effects (font (size 1.27 1.27)) (justify left bottom))
   )
+  (label "PROG_NMI" (at 111.125 57.15 0)
+    (effects (font (size 1.27 1.27)) (justify left bottom))
+  )

Commit message: Re-route complete
Parts:
- added R10, R11, R12, R13, R14, R15, R16, R17, R18, R19, R20, R4, R5, R6, R7, R8, R9: 10kΩ, Resistor_THT:R_Axial_DIN0207_L6.3mm_D2.5mm_P10.16mm_Horizontal, symbol Device:R_Small_US
- X1: footprint OST_USB-B1HSB6 -> USB-B1HSB6:OST_USB-B1HSB6
Connections:
- net GND: now also U1.30 (p2,2/intp1), U1.31 (p2,3/intp2/ci), U1.32 (p2,4/intp3), U1.33 (p2,5/intp4/asck), U1.34 (p2,6/intp5), U1.35 (p2,7/si), U1.8 (X1), R10.2, R11.2, R12.2, R13.2, R14.2, R15.2, R16.2, R17.2, R18.2, R19.2, R20.2, R4.1, R5.2, R6.2, R7.2, R8.2, R9.2; no longer U1.42 (AVss)
- net PROG_A9: now also U1.29 (p2,1/intp0); no longer U1.16 (p5,1/a9)
- net PROG_NMI: now also J1.20 (Pin_20); no longer J1.22 (Pin_22)
- net PROG_A15: now reaches U1.10 (p5,7/a15)
- net PROG_A15: now also J1.22 (Pin_22)
- net at U1.2 (p6,3/a19): now also R13.1
- net at U1.3 (p6,2/a18): now also R12.1
- net at U1.38 (p3,2/sck): now also R9.1
- net at U1.39 (p3,3/so/sb0): now also R7.1
- net at U1.4 (p6,1/a17): now also R11.1
- net at U1.43 (AVref): now also R5.1
- net at U1.44 (p7,5/AN5): now also R14.1
- net at U1.45 (p7,4/AN4): now also R17.1
- net at U1.46 (p7,3/AN3): now also R19.1
- net at U1.47 (p7,2/AN2): now also R16.1
- net at U1.48 (p7,1/AN1): now also R8.1
- net at U1.49 (p7,0/AN0): now also R6.1
- net at U1.5 (p6,0/a16): now also R10.1
- net at U1.62 (p6,7/~{REFRQ}/AN7): now also R15.1
- net at U1.63 (p6,6/~{WAIT}/AN6): now also R18.1
- new net: R20.1, U1.16 (p5,1/a9)
- new net: R4.2, U1.42 (AVss)
- no-connect marks 7 -> 14
Other:
- note added: "TODO: Double check where A9 lives"
- note added: "TODO: Recheck this"
