File: upd78214-arduino-mega-hat/upd78214-arduino-mega-hat.kicad_pcb (KiCad board)
At the start: 4 copper layers, 101.6 x 53.3 mm, 19 parts, among them J1 Power, J2 PWM, J3 Analog, J4 PWM, J5 Analog, J6 Communication, J7 Digital, U1 upd78214-64p-qfp, Y1 4-12MHz

Commit message: Correct Shield to use right footprint, have jumper pins
Parts:
- added J8: NMI +12V / GND, Connector_PinHeader_2.54mm:PinHeader_1x02_P2.54mm_Vertical, F.Cu at (150.7, 66.5)
- U1: footprint Package_QFP:TQFP-64_14x14mm_P0.8mm -> NEC:QFP-64_14x14_Pitch0.8mm
Connections:
- U1 pad 28: unconnected-(U1-p2,0/nmi-Pad28) -> /NMI
Routing:
- net /NMI: track 0.00 -> 19.0 mm
- net Net-(U1-X1): track 16.6 -> 28.7 mm
- net /a9: track 82.5 -> 89.5 mm
- net /a13: track 84.3 -> 91.1 mm
- net /a12: track 83.2 -> 90.0 mm
- net /a14: track 84.0 -> 90.8 mm
- net /a11: track 83.3 -> 89.9 mm
- net /a10: track 83.4 -> 89.8 mm
- net /a15: track 84.3 -> 90.6 mm
- net /ad2: track 56.8 -> 62.5 mm
- net /ad3: track 58.8 -> 64.3 mm
- net /ad1: track 56.0 -> 61.4 mm
- net /ad0: track 55.8 -> 60.7 mm
- net /ad4: track 58.5 -> 61.5 mm
- net /ad6: track 60.5 -> 63.6 mm, vias 0 -> 1
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Other:
- board text added: "Apply +12V here: 1 = NMI, 2 = GND"
